Commit message: Extend gripper fingers 9cm, parametrize gazebo namespace, add human-friendly controllers
- franka_hand.xacro: tcp_xyz default 0.1034 -> 0.1934, add finger_extension_m
  param with matching collision geometry for the extended fingers
- panda.launch/robot.launch: expose finger_extension_m, tcp_xyz, and
  gazebo_namespace as top-level launch args (roslaunch's arg:=value parsing
  breaks on a value that itself contains ":=", so these can't be folded into
  xacro_args; spawn_model's gazebo_namespace default also doesn't follow an
  outer namespace group)
- Add franka_human_friendly_controllers package
- Misc controller launch/rviz tweaks

Co-Authored-By: Claude Sonnet 5 <noreply@anthropic.com>
Claude-Session: https://claude.ai/code/session_0176nUydYKQzSK2UarpXgR7G

File: franka_description/robots/common/franka_hand.xacro (robot description, xacro)
@@ -2,5 +2,5 @@
 <robot xmlns:xacro="http://www.ros.org/wiki/xacro" name="hand">
   <!-- safety_distance: Minimum safety distance in [m] by which the collision volumes are expanded and which is enforced during robot motions -->
-  <xacro:macro name="franka_hand" params="connected_to:='' arm_id:='panda' rpy:='0 0 0' xyz:='0 0 0' tcp_xyz:='0 0 0.1034' tcp_rpy:='0 0 0' safety_distance:=0 gazebo:=false description_pkg:=franka_description">
+  <xacro:macro name="franka_hand" params="connected_to:='' arm_id:='panda' rpy:='0 0 0' xyz:='0 0 0' tcp_xyz:='0 0 0.1934' tcp_rpy:='0 0 0' safety_distance:=0 gazebo:=false description_pkg:=franka_description finger_extension_m:=0.09">
     <xacro:unless value="${connected_to == ''}">
       <joint name="${arm_id}_hand_joint" type="fixed">
@@ -57,4 +57,15 @@
         </geometry>
       </collision>
+      <!-- Finger extension: length is parametrized (finger_extension_m, default 0.09 to
+           match the original hardcoded 9cm piece this replaces); anchored so its proximal
+           end stays flush against the rubber tip block above (which ends at z=54.5e-3)
+           regardless of length, and its distal end tracks tcp_xyz's z (see franka_robot.xacro:
+           tcp_z = 0.1034 [stock fingertip] + finger_extension_m). -->
+      <collision>
+        <origin xyz="0 7.58e-3 ${54.5e-3 + finger_extension_m/2}" rpy="0 0 0" />
+        <geometry>
+          <box size="17.5e-3 15.2e-3 ${finger_extension_m}" />
+        </geometry>
+      </collision>
       <xacro:if value="${gazebo}">
         <xacro:inertial_props name="leftfinger" />
@@ -96,4 +107,11 @@
         </geometry>
       </collision>
+      <!-- Finger extension: see leftfinger's matching block above for the parametrization. -->
+      <collision>
+        <origin xyz="0 -7.58e-3 ${54.5e-3 + finger_extension_m/2}" rpy="0 0 0" />
+        <geometry>
+          <box size="17.5e-3 15.2e-3 ${finger_extension_m}" />
+        </geometry>
+      </collision>
       <xacro:if value="${gazebo}">
         <xacro:inertial_props name="rightfinger" />

File: franka_description/robots/common/franka_robot.xacro (robot description, xacro)
@@ -5,8 +5,14 @@
     <!-- Should a franka_gripper be mounted at the flange?" -->
     <xacro:arg name="hand" default="false" />
-    <!-- Positional offset between $(arm_id)_hand -> $(arm_id)_hand_tcp [m]. Only used when hand:=true -->
-    <xacro:arg name="tcp_xyz" default="0 0 0.1034" />
+    <!-- Positional offset between $(arm_id)_hand -> $(arm_id)_hand_tcp [m]. Only used when hand:=true.
+         z should track finger_extension_m below: 0.1034 (stock fingertip, no extension) + finger_extension_m. -->
+    <xacro:arg name="tcp_xyz" default="0 0 0.1934" />
     <!-- Rotational offset between $(arm_id)_hand -> $(arm_id)_hand_tcp [rad]. Only used when hand:=true -->
     <xacro:arg name="tcp_rpy" default="0 0 0" />
+    <!-- Length of the custom finger-extension collision box [m]. Only used when hand:=true.
+         Default 0.09 matches this project's original hardcoded 9cm extension; override together
+         with tcp_xyz (see above) to test other finger lengths without editing this file, e.g. for
+         a 6cm extension: finger_extension_m:=0.06 tcp_xyz:="0 0 0.1634" -->
+    <xacro:arg name="finger_extension_m" default="0.09" />
     <!-- Is the robot being simulated in gazebo?" -->
     <xacro:arg name="gazebo" default="false" />
@@ -28,4 +34,5 @@
           safety_distance="0.03"
           gazebo="$(arg gazebo)"
+          finger_extension_m="$(arg finger_extension_m)"
        />
     </xacro:if>
